Commit message: feat: wheels added in xacro

File: xacro/my-jetbot.xacro (robot description, xacro)
@@ -11,5 +11,5 @@
     name = "base"
     parent = "odom"
-    joint_origin_xyz = "0 0 0.0445"
+    joint_origin_xyz = "0 0 0"
 />
 <xacro:standoff
@@ -51,3 +51,51 @@
     joint_origin_xyz = "-0.06277 -0.04275 0.02125"
 />
+<xacro:standoff
+    name ="standoff5"
+    radius = "0.0025"
+    length = "0.081"
+    mass = "0.5"
+    parent = "level2_link"
+    joint_origin_xyz = "-0.06277 0.042975 0.01975"
+/>
+<xacro:standoff
+    name ="standoff6"
+    radius = "0.0025"
+    length = "0.081"
+    mass = "0.5"
+    parent = "level2_link"
+    joint_origin_xyz = "0.06277 0.042975 0.01975"
+/>
+<xacro:standoff
+    name ="standoff7"
+    radius = "0.0025"
+    length = "0.081"
+    mass = "0.5"
+    parent = "level2_link"
+    joint_origin_xyz = "0.06277 -0.042975 0.01975"
+/>
+<xacro:standoff
+    name ="standoff8"
+    radius = "0.0025"
+    length = "0.081"
+    mass = "0.5"
+    parent = "level2_link"
+    joint_origin_xyz = "-0.06277 -0.042975 0.01975"
+/>
+<!-- level 3 -->
+<xacro:base-plate
+    name = "level3"
+    parent = "standoff6"
+    joint_origin_xyz = "-0.06277 -0.04275 0.039"
+/>
+<xacro:wheel
+    name = "left_wheel"
+    parent = "base_link"
+    joint_origin_xyz = "0.047135 0.05625 0.008125"
+/>
+<xacro:wheel
+    name = "right_wheel"
+    parent = "base_link"
+    joint_origin_xyz = "0.047135 -0.05625 0.008125"
+/>
 </robot>

File: xacro/wheel.xacro (robot description, xacro)
@@ -1,34 +1,15 @@
 <?xml version="1.0"?>
 <robot xmlns:xacro="http://www.ros.org/wiki/xacro" name="wheel">
-    <!--
-      <link name="left_wheel">
-        <visual>
-          <origin xyz="0 0 0" rpy="0 0 0"/>
-          <geometry>
-            <cylinder radius="0.03" length="0.01"/>
-          </geometry>
-          <material name="black">
-            <color rgba="0.0 0.0 0.0 1.0"/>
-          </material>
-        </visual>
-        <collision>
-          <origin xyz="0 0 0" rpy="0 0 0"/>
-          <geometry>
-            <cylinder radius="0.03" length="0.01"/>
-          </geometry>
-        </collision>
-      </link>
-    -->
     <xacro:macro name="wheel" params="name parent joint_origin_xyz">
         <link name="${name}_link">
             <inertial>
-                <origin rpy="0 0 0" xyz="0 0 0"/>
+                <origin rpy="0 1.5707 1.5707" xyz="0 0 0"/>
                 <mass value="0.1"/>
                 <inertia ixx="0.001" ixy="0.0" ixz="0.0" iyy="0.001" iyz="0.0" izz="0.001"/>
             </inertial>
             <visual>
-                <origin rpy="0 0 0" xyz="0 0 0"/>
+                <origin rpy="0 1.5707 1.5707" xyz="0 0 0"/>
                 <geometry>
-                    <cylinder length="0.01" radius="0.03"/>
+                    <cylinder length="0.026" radius="0.0325"/>
                 </geometry>
             </visual>
@@ -36,5 +17,5 @@
                 <origin rpy="0 1.5707 1.5707" xyz="0 0 0"/>
                 <geometry>
-                    <cylinder length="${length}" radius="${radius}"/>
+                    <cylinder length="0.026" radius="0.0325"/>
                 </geometry>
             </collision>
@@ -45,5 +26,5 @@
             <mu1>10.0</mu1>
             <mu2>10.0</mu2>
-            <material>${material}</material>
+            <material>Gazebo/Yellow</material>
         </gazebo>
         <joint name="${name}_joint" type="continuous">

Commit message: feat: adding back caster

File: xacro/my-jetbot.xacro (robot description, xacro)
@@ -1,101 +1,182 @@
 <?xml version="1.0"?>
-<robot xmlns:xacro="http://www.ros.org/wiki/xacro" name="jetbot">
-<xacro:include filename="$(find jetbot_sim)/xacro/standoff.xacro"/>
-<xacro:include filename="$(find jetbot_sim)/xacro/wheel.xacro"/>
-<xacro:include filename="$(find jetbot_sim)/xacro/base-plate.xacro"/>
-<xacro:property name="include_laser" value="true" />
-<!-- odom, so base_link can have inertia -->
-<link name="odom"/>
-<!-- robot base -->
-<xacro:base-plate
-    name = "base"
-    parent = "odom"
-    joint_origin_xyz = "0 0 0.043"
-/>
-<xacro:standoff
-    name ="standoff1"
-    radius = "0.0025"
-    length = "0.0393"
-    mass = "0.5"
-    parent = "base_link"
-    joint_origin_xyz = "-0.06277 0.042975 0.01975"
-/>
-<xacro:standoff
-    name ="standoff2"
-    radius = "0.0025"
-    length = "0.0393"
-    mass = "0.5"
-    parent = "base_link"
-    joint_origin_xyz = "0.06277 0.042975 0.01975"
-/>
-<xacro:standoff
-    name ="standoff3"
-    radius = "0.0025"
-    length = "0.0393"
-    mass = "0.5"
-    parent = "base_link"
-    joint_origin_xyz = "0.06277 -0.042975 0.01975"
-/>
-<xacro:standoff
-    name ="standoff4"
-    radius = "0.0025"
-    length = "0.0393"
-    mass = "0.5"
-    parent = "base_link"
-    joint_origin_xyz = "-0.06277 -0.042975 0.01975"
-/>
-<!-- level 2 -->
-<xacro:base-plate
-    name = "level2"
-    parent = "standoff2"
-    joint_origin_xyz = "-0.06277 -0.04275 0.02125"
-/>
-<xacro:standoff
-    name ="standoff5"
-    radius = "0.0025"
-    length = "0.081"
-    mass = "0.5"
-    parent = "level2_link"
-    joint_origin_xyz = "-0.06277 0.042975 0.01975"
-/>
-<xacro:standoff
-    name ="standoff6"
-    radius = "0.0025"
-    length = "0.081"
-    mass = "0.5"
-    parent = "level2_link"
-    joint_origin_xyz = "0.06277 0.042975 0.01975"
-/>
-<xacro:standoff
-    name ="standoff7"
-    radius = "0.0025"
-    length = "0.081"
-    mass = "0.5"
-    parent = "level2_link"
-    joint_origin_xyz = "0.06277 -0.042975 0.01975"
-/>
-<xacro:standoff
-    name ="standoff8"
-    radius = "0.0025"
-    length = "0.081"
-    mass = "0.5"
-    parent = "level2_link"
-    joint_origin_xyz = "-0.06277 -0.042975 0.01975"
-/>
-<!-- level 3 -->
-<xacro:base-plate
-    name = "level3"
-    parent = "standoff6"
-    joint_origin_xyz = "-0.06277 -0.04275 0.039"
-/>
-<xacro:wheel
-    name = "left_wheel"
-    parent = "base_link"
-    joint_origin_xyz = "0.047135 0.0625 -0.008125"
-/>
-<xacro:wheel
-    name = "right_wheel"
-    parent = "base_link"
-    joint_origin_xyz = "0.047135 -0.0625 -0.008125"
-/>
+    <robot xmlns:xacro="http://www.ros.org/wiki/xacro" name="jetbot">
+    <xacro:include filename="$(find jetbot_sim)/xacro/standoff.xacro"/>
+    <xacro:include filename="$(find jetbot_sim)/xacro/wheel.xacro"/>
+    <xacro:include filename="$(find jetbot_sim)/xacro/base-plate.xacro"/>
+    <xacro:property name="include_laser" value="true" />
+    <!-- odom, so base_link can have inertia -->
+    <link name="odom"/>
+    <!-- robot base -->
+    <xacro:base-plate
+        name = "base"
+        parent = "odom"
+        joint_origin_xyz = "0 0 0.043"
+    />
+    <xacro:standoff
+        name ="standoff1"
+        radius = "0.0025"
+        length = "0.0393"
+        mass = "0.5"
+        parent = "base_link"
+        joint_origin_xyz = "-0.06277 0.042975 0.01975"
+    />
+    <xacro:standoff
+        name ="standoff2"
+        radius = "0.0025"
+        length = "0.0393"
+        mass = "0.5"
+        parent = "base_link"
+        joint_origin_xyz = "0.06277 0.042975 0.01975"
+    />
+    <xacro:standoff
+        name ="standoff3"
+        radius = "0.0025"
+        length = "0.0393"
+        mass = "0.5"
+        parent = "base_link"
+        joint_origin_xyz = "0.06277 -0.042975 0.01975"
+    />
+    <xacro:standoff
+        name ="standoff4"
+        radius = "0.0025"
+        length = "0.0393"
+        mass = "0.5"
+        parent = "base_link"
+        joint_origin_xyz = "-0.06277 -0.042975 0.01975"
+    />
+    <!-- level 2 -->
+    <xacro:base-plate
+        name = "level2"
+        parent = "standoff2"
+        joint_origin_xyz = "-0.06277 -0.04275 0.02125"
+    />
+    <xacro:standoff
+        name ="standoff5"
+        radius = "0.0025"
+        length = "0.081"
+        mass = "0.5"
+        parent = "level2_link"
+        joint_origin_xyz = "-0.06277 0.042975 0.01975"
+    />
+    <xacro:standoff
+        name ="standoff6"
+        radius = "0.0025"
+        length = "0.081"
+        mass = "0.5"
+        parent = "level2_link"
+        joint_origin_xyz = "0.06277 0.042975 0.01975"
+    />
+    <xacro:standoff
+        name ="standoff7"
+        radius = "0.0025"
+        length = "0.081"
+        mass = "0.5"
+        parent = "level2_link"
+        joint_origin_xyz = "0.06277 -0.042975 0.01975"
+    />
+    <xacro:standoff
+        name ="standoff8"
+        radius = "0.0025"
+        length = "0.081"
+        mass = "0.5"
+        parent = "level2_link"
+        joint_origin_xyz = "-0.06277 -0.042975 0.01975"
+    />
+    <!-- level 3 -->
+    <xacro:base-plate
+        name = "level3"
+        parent = "standoff6"
+        joint_origin_xyz = "-0.06277 -0.04275 0.039"
+    />
+    <xacro:wheel
+        name = "left_wheel"
+        parent = "base_link"
+        joint_origin_xyz = "0.047135 0.0625 -0.008125"
+    />
+    <xacro:wheel
+        name = "right_wheel"
+        parent = "base_link"
+        joint_origin_xyz = "0.047135 -0.0625 -0.008125"
+    />
+    <xacro:standoff
+        name = "standoff9"
+        radius = "0.0025"
+        length = "0.0245"
+        mass = "0.1"
+        parent = "base_link"
+        joint_origin_xyz = "-0.05477 0.02 -0.01375"
+    />
+    <xacro:standoff
+        name = "standoff10"
+        radius = "0.0025"
+        length = "0.0245"
+        mass = "0.1"
+        parent = "base_link"
+        joint_origin_xyz = "-0.05477 -0.02 -0.01375"
+    />
+    <link name="caster_plate_link">
+        <visual>
+          <geometry>
+            <box size="0.023 0.05 0.008"/>
+          </geometry>
+        </visual>
+        <collision>
+          <geometry>
+            <box size="0.023 0.01 0.008"/>
+          </geometry>
+        </collision>
+        <inertial>
+          <mass value="0.5"/>
+          <origin rpy="0 0 0" xyz="0 0 0"/>
+          <inertia ixx="0.0008333333333333335" ixy="0" ixz="0" iyy="0.0008333333333333335" iyz="0" izz="0.0008333333333333335"/>
+        </inertial>
+    </link>
+    <joint name="caster_plate_joint" type="fixed">
+        <origin rpy="0 0 0" xyz="0 0.02 -0.0165" />
+        <parent link="standoff10" />
+        <child link="caster_plate_link" />
+    </joint>
+    <link name="caster_ball_link">
+        <visual>
+          <origin xyz="0 0 0" rpy="0 0 0"/>
+          <geometry>
+            <sphere radius="0.0075"/>
+          </geometry>
+          <material name="silver">
+            <color rgba="0.75 0.75 0.75 1.0"/>
+          </material>
+        </visual>
+        <collision>
+          <origin xyz="0 0 0" rpy="0 0 0"/>
+          <geometry>
+            <sphere radius="0.0075"/>
+          </geometry>
+        </collision>
+        <inertial>
+          <mass value="0.01"/>
+          <origin xyz="0 0 0" rpy="0 0 0"/>
+          <inertia ixx="0.00001" ixy="0.0" ixz="0.0" iyy="0.00001" iyz="0.0" izz="0.00001"/>
+        </inertial>
+    </link>
+    <joint name="caster_ball_roll_joint" type="continuous">
+        <parent link="caster_plate_link"/>
+        <child link="caster_ball_link"/>
+        <!-- <origin rpy="0 0 0" xyz="-0.055 0 -0.0115"/> -->
+        <origin rpy="0 0 0" xyz="0 0 -0.0115"/>
+        <axis xyz="1 0 0" />
+    </joint>
+    <link name="caster_ball_pitch_link" />
+    <joint name="caster_ball_pitch_joint" type="continuous">
+        <parent link="caster_ball_link"/>
+        <child link="caster_ball_pitch_link"/>
+        <origin xyz="0 0 0" rpy="0 0 0"/>
+        <axis xyz="0 1 0"/>
+    </joint>
+    <link name="caster_ball_yaw_link" />
+    <joint name="caster_ball_yaw_joint" type="continuous">
+        <parent link="caster_ball_pitch_link"/>
+        <child link="caster_ball_yaw_link"/>
+        <origin xyz="0 0 0" rpy="0 0 0"/>
+        <axis xyz="0 0 1"/>
+    </joint>
 </robot>
