Commit message: feat: added lidar to model

File: xacro/laser-scanner.xacro (robot description, xacro)
@@ -1,32 +1,29 @@
 <?xml version="1.0"?>
-<robot xmlns:xacro="http://www.ros.org/wiki/xacro" name="laser_scanner">
-  <xacro:macro name="laser_scanner">
-    <xacro:arg name="include_laser" default="true"/>
-    <xacro:if value="${include_laser}">
-        <link name="hokuyo_link"> <!-- aka laser_scan_link -->
+<robot xmlns:xacro="http://www.ros.org/wiki/xacro" name="ydlidar">
+  <xacro:macro name="ydlidar" params="name package parent joint_origin_xyz">
+        <link name="${name}_link">
             <visual>
-            <origin rpy="0 0 0" xyz="0.03 0 0.003"/>
-            <geometry>
-                <mesh filename="package://barista_robot_description/meshes/hokuyo_urg_04lx.dae" />
-            </geometry>
+                <origin rpy="0 0 0" xyz="0 0 0"/>
+                <geometry>
+                    <mesh filename="package://${package}/meshes/hokuyo_urg_04lx.dae" />
+                </geometry>
             </visual>
             <inertial>
-            <!-- from https://www.hokuyo-aut.jp/dl/Specifications_URG-04LX_1513063395.pdf -->
-            <mass value="0.16"/>
-            <inertia ixx="1.0" ixy="0.0" ixz="0.0" iyy="1.0" iyz="0.0" izz="1.0"/>
+                <mass value="0.16"/>
+                <inertia ixx="1.0" ixy="0.0" ixz="0.0" iyy="1.0" iyz="0.0" izz="1.0"/>
             </inertial>
             <collision>
-            <origin xyz="0 0 0" rpy="0 0 0" />
-            <geometry>
-                <mesh filename="package://barista_robot_description/meshes/hokuyo_urg_04lx.stl" />
-            </geometry>
+                <origin xyz="0 0 0" rpy="0 0 0" />
+                <geometry>
+                    <mesh filename="package://${package}/meshes/hokuyo_urg_04lx.stl" />
+                </geometry>
             </collision>
         </link>
-        <joint name="hokuyo_joint" type="fixed"> <!-- aka laser_scan_link_joint-->
-            <parent link="base_link"/>
-            <child link="hokuyo_link"/>
-            <origin xyz="0.1 0 0.08" rpy="0 0 1.5707" />
+        <joint name="${name}_joint" type="fixed">
+            <parent link="${parent}"/>
+            <child link="${name}_link"/>
+            <origin rpy="0 0 0"  xyz="${joint_origin_xyz}" />
         </joint>
-        <gazebo reference="hokuyo_link">
+        <gazebo reference="${name}_link">
             <sensor name="head_hokuyo_sensor" type="ray">
             <pose>0 0 0 0 0 0</pose>
@@ -63,5 +60,4 @@
             </sensor>
         </gazebo>
-    </xacro:if>
   </xacro:macro>
   </robot>

File: xacro/my-jetbot.xacro (robot description, xacro)
@@ -4,5 +4,5 @@
     <xacro:include filename="$(find jetbot_sim)/xacro/wheel.xacro"/>
     <xacro:include filename="$(find jetbot_sim)/xacro/base-plate.xacro"/>
-    <xacro:property name="include_laser" value="true" />
+    <xacro:include filename="$(find jetbot_sim)/xacro/laser-scanner.xacro"/>
     <!-- odom, so base_link can have inertia -->
     <link name="odom"/>
@@ -180,3 +180,9 @@
         <axis xyz="0 0 1"/>
     </joint>
+    <xacro:ydlidar
+        name = "ydlidar"
+        package = "jetbot_sim"
+        parent = "level3_link"
+        joint_origin_xyz = "0 0 0.0015"
+    />
 </robot>

File: xacro/standoff.xacro (robot description, xacro)
@@ -1,4 +1,4 @@
 <?xml version="1.0"?>
-<robot xmlns:xacro="http://www.ros.org/wiki/xacro" name="base-plate">
+<robot xmlns:xacro="http://www.ros.org/wiki/xacro" name="standoff">
     <xacro:macro name="standoff" params="name radius length mass parent joint_origin_xyz">
        <link name="${name}">

Commit message: feat adding basic geometry for the camera and IMU

File: xacro/laser-scanner.xacro (robot description, xacro)
@@ -6,6 +6,10 @@
                 <origin rpy="0 0 0" xyz="0 0 0"/>
                 <geometry>
-                    <mesh filename="package://${package}/meshes/hokuyo_urg_04lx.dae" />
+                    <mesh
+                            filename="package://${package}/meshes/hokuyo_urg_04lx.dae"
+                            scale = "0.8 0.8 0.8"
+                    />
                 </geometry>
+                <material name="Gazebo/Blue"/>
             </visual>
             <inertial>
@@ -16,5 +20,8 @@
                 <origin xyz="0 0 0" rpy="0 0 0" />
                 <geometry>
-                    <mesh filename="package://${package}/meshes/hokuyo_urg_04lx.stl" />
+                    <mesh
+                            filename="package://${package}/meshes/hokuyo_urg_04lx.stl"
+                            scale = "0.3 0.3 0.3"
+                    />
                 </geometry>
             </collision>
@@ -26,4 +33,5 @@
         </joint>
         <gazebo reference="${name}_link">
+            <material>Gazebo/Blue</material>
             <sensor name="head_hokuyo_sensor" type="ray">
             <pose>0 0 0 0 0 0</pose>

File: xacro/my-jetbot.xacro (robot description, xacro)
@@ -1,8 +1,10 @@
 <?xml version="1.0"?>
-    <robot xmlns:xacro="http://www.ros.org/wiki/xacro" name="jetbot">
+<robot xmlns:xacro="http://www.ros.org/wiki/xacro" name="jetbot">
     <xacro:include filename="$(find jetbot_sim)/xacro/standoff.xacro"/>
     <xacro:include filename="$(find jetbot_sim)/xacro/wheel.xacro"/>
     <xacro:include filename="$(find jetbot_sim)/xacro/base-plate.xacro"/>
     <xacro:include filename="$(find jetbot_sim)/xacro/laser-scanner.xacro"/>
+    <xacro:include filename="$(find jetbot_sim)/xacro/camera.xacro"/>
+    <xacro:include filename="$(find jetbot_sim)/xacro/imu.xacro"/>
     <!-- odom, so base_link can have inertia -->
     <link name="odom"/>
@@ -186,3 +188,15 @@
         joint_origin_xyz = "0 0 0.0015"
     />
+    <xacro:camera
+        name = "front_camera"
+        parent = "level2_link"
+        joint_origin_xyz = "0 0 0"
+        joint_origin_rpy = "0 0 0"
+    />
+    <xacro:imu
+        name = "default"
+        parent = "level3_link"
+        joint_origin_xyz = "0 -0.03975 0.02"
+        joint_origin_rpy = "0 0 0"
+    />
 </robot>
