Commit message: fix: adding front camera

File: xacro/camera.xacro (robot description, xacro)
@@ -1,9 +1,9 @@
 <robot xmlns:xacro="http://www.ros.org/wiki/xacro" name="camera">
     <xacro:macro name="camera" params="name parent joint_origin_xyz joint_origin_rpy">
-        <link name="${name}_camera_link">
+        <link name="${name}_camera_board_link">
             <visual>
                 <origin xyz="0 0 0" rpy="0 0 0"/>
                 <geometry>
-                    <box size="0.04 0.04 0.02"/>
+                    <box size="0.025 0.025 0.001"/>
                 </geometry>
                 <material name="black">
@@ -14,5 +14,5 @@
                 <origin xyz="0 0 0" rpy="0 0 0"/>
                 <geometry>
-                    <box size="0.04 0.04 0.02"/>
+                    <box size="0.025 0.025 0.001"/>
                 </geometry>
             </collision>
@@ -23,9 +23,60 @@
             </inertial>
         </link>
-        <joint name="${name}_camera_joint" type="fixed">
+        <joint name="${name}_camera_board_joint" type="fixed">
             <parent link="${parent}"/>
-            <child link="${name}_camera_link"/>
-            <origin rpy="${joint_origin_rpy}" xyz="${joint_origin_xyz}" />
+            <child link="${name}_camera_board_link"/>
+            <origin rpy="${joint_origin_rpy}" xyz="${joint_origin_xyz}"/>
         </joint>
+        <gazebo reference="${name}_camera_board_link">
+            <material>Gazebo/Gold</material>
+        </gazebo>
+        <link name="${name}_camera_bottom_link">
+            <inertial>
+                <mass value="0.1"/>
+                <inertia ixx="0.001" ixy="0.0" ixz="0.0" iyy="0.001" iyz="0.0" izz="0.001"/>
+            </inertial>
+            <visual>
+                <geometry>
+                    <cylinder length="0.01" radius="0.0045"/>
+                </geometry>
+            </visual>
+            <collision>
+                <geometry>
+                    <cylinder length="0.01" radius="0.0045"/>
+                </geometry>
+            </collision>
+        </link>
+        <joint name="${name}_camera_bottom_joint" type="fixed">
+            <origin rpy="0 0 0" xyz="0 0 -0.005"/>
+            <parent link="${name}_camera_board_link"/>
+            <child link="${name}_camera_bottom_link"/>
+        </joint>
+        <gazebo reference="${name}_camera_bottom_link">
+            <material>Gazebo/Black</material>
+        </gazebo>
+        <link name="${name}_camera_top_link">
+            <inertial>
+                <mass value="0.1"/>
+                <inertia ixx="0.001" ixy="0.0" ixz="0.0" iyy="0.001" iyz="0.0" izz="0.001"/>
+            </inertial>
+            <visual>
+                <geometry>
+                    <cylinder length="0.0045" radius="0.006"/>
+                </geometry>
+            </visual>
+            <collision>
+                <geometry>
+                    <cylinder length="0.0045" radius="0.006"/>
+                </geometry>
+            </collision>
+        </link>
+        <joint name="${name}_camera_top_joint" type="fixed">
+            <origin rpy="0 0 0" xyz="0 0 -0.0075"/>
+            <parent link="${name}_camera_bottom_link"/>
+            <child link="${name}_camera_top_link"/>
+        </joint>
+        <gazebo reference="${name}_camera_top_link">
+            <material>Gazebo/Black</material>
+        </gazebo>
         <gazebo>
             <plugin name="camera_controller" filename="libgazebo_ros_camera.so">

File: xacro/imu.xacro (robot description, xacro)
@@ -7,5 +7,5 @@
                 <origin xyz="0 0 0" rpy="0 0 0"/>
                 <geometry>
-                    <box size="0.02 0.01 0.003"/>
+                    <box size="0.026 0.0155 0.002"/>
                 </geometry>
             </visual>
@@ -13,5 +13,5 @@
                 <origin xyz="0 0 0" rpy="0 0 0"/>
                 <geometry>
-                    <box size="0.02 0.01 0.003"/>
+                    <box size="0.026 0.0155 0.002"/>
                 </geometry>
             </collision>

File: xacro/my-jetbot.xacro (robot description, xacro)
@@ -190,5 +190,5 @@
         joint_origin_xyz = "-0.05977 -0.0315 0.018"
     />
-        <xacro:standoff
+    <xacro:standoff
         name = "standoff12"
         radius = "0.0025"
@@ -198,5 +198,5 @@
         joint_origin_xyz = "-0.05977 0.0315 0.018"
     />
-        <xacro:standoff
+    <xacro:standoff
         name = "standoff13"
         radius = "0.0025"
@@ -214,13 +214,38 @@
         joint_origin_xyz = "-0.00477 0.0315 0.018"
     />
-        <xacro:ydlidar
+    <xacro:ydlidar
         name = "primary"
         parent = "standoff14"
         joint_origin_xyz = "-0.01 -0.032 0.0215"
     />
+    <link name="camera_plate_link">
+        <visual>
+          <geometry>
+            <box size="0.022 0.072 0.003"/>
+          </geometry>
+        </visual>
+        <collision>
+          <geometry>
+            <box size="0.022 0.072 0.003"/>
+          </geometry>
+        </collision>
+        <inertial>
+          <mass value="0.5"/>
+          <origin rpy="0 0 0" xyz="0 0 0"/>
+          <inertia ixx="0.0008333333333333335" ixy="0" ixz="0" iyy="0.0008333333333333335" iyz="0" izz="0.0008333333333333335"/>
+        </inertial>
+    </link>
+    <joint name="camera_plate_joint" type="fixed">
+        <origin rpy="0 -1 0" xyz="0.075 0 0.01" />
+        <parent link="level2_link" />
+        <child link="camera_plate_link" />
+      </joint>
+      <gazebo reference="camera_plate_link">
+        <material>Gazebo/Black</material>
+      </gazebo>
     <xacro:camera
         name = "front_camera"
-        parent = "level2_link"
-        joint_origin_xyz = "0 0 0"
+        parent = "camera_plate_link"
+        joint_origin_xyz = "0 -0.018 -0.002"
         joint_origin_rpy = "0 0 0"
     />

File: xacro/wheel.xacro (robot description, xacro)
@@ -21,5 +21,5 @@
             </collision>
         </link>
-        <gazebo reference="${name}">
+        <gazebo reference="${name}_link">
             <kp>1000000000000000000000000000.0</kp>
             <kd>1000000000000000000000000000.0</kd>
