Commit message: feat: xacro working

File: xacro/base-plate.xacro (robot description, xacro)
@@ -1,5 +1,5 @@
 <?xml version="1.0"?>
 <robot xmlns:xacro="http://www.ros.org/wiki/xacro" name="base-plate">
-    <xacro:macro name="wheel" params="name parent joint_origin_xyz">
+    <xacro:macro name="base-plate" params="name parent joint_origin_xyz">
         <link name="${name}_link">
         <visual>

File: xacro/my-jetbot.xacro (robot description, xacro)
@@ -1,360 +1,53 @@
 <?xml version="1.0"?>
-<robot xmlns:xacro="http://www.ros.org/wiki/xacro" name="barista_bot">
-<xacro:include filename="$(find barista_robot_description)/xacro/standoff.xacro"/>
-<xacro:include filename="$(find barista_robot_description)/xacro/wheel.xacro"/>
-<xacro:include filename="$(find barista_robot_description)/xacro/cup_holder_tray.xacro"/>
-<xacro:include filename="$(find barista_robot_description)/xacro/laser_scanner.xacro"/>
+<robot xmlns:xacro="http://www.ros.org/wiki/xacro" name="jetbot">
+<xacro:include filename="$(find jetbot_sim)/xacro/standoff.xacro"/>
+<xacro:include filename="$(find jetbot_sim)/xacro/wheel.xacro"/>
+<xacro:include filename="$(find jetbot_sim)/xacro/base-plate.xacro"/>
 <xacro:property name="include_laser" value="true" />
 <!-- odom, so base_link can have inertia -->
 <link name="odom"/>
-<joint name="base_link_base" type="fixed">
-  <origin rpy="0 0 0" xyz="0 0 0" />
-  <parent link="odom" />
-  <child link="base_link" />
-</joint>
 <!-- robot base -->
-  <link name="base_link">
-    <visual>
-      <geometry>
-        <cylinder radius="0.178" length="0.155" />
-      </geometry>
-    </visual>
-    <collision>
-      <geometry>
-        <cylinder radius="0.178" length="0.155" />
-      </geometry>
-    </collision>
-    <inertial>
-      <mass value="0.5"/>
-      <origin rpy="0 0 0" xyz="0 0 0"/>
-      <inertia ixx="0.0008333333333333335" ixy="0" ixz="0" iyy="0.0008333333333333335" iyz="0" izz="0.0008333333333333335"/>
-    </inertial>
-  </link>
-  <gazebo reference="base_link">
-    <material>Gazebo/Black</material>
-  </gazebo>
- <!-- standoffs -->
-  <xacro:standoff name="standoff1"
-    radius="0.01"
-    length="0.22"
-    mass="0.5"
-    material="Gazebo/Gold"
-    parent="base_link"
-    joint_origin_xyz="0.0375 0.1 0.185"
-  />
-  <xacro:standoff name="standoff2"
-    radius="0.01"
-    length="0.22"
-    mass="0.5"
-    material="Gazebo/Gold"
-    parent="base_link"
-    joint_origin_xyz="-0.0375 0.1 0.185"
-  />
-  <xacro:standoff name="standoff3"
-    radius="0.01"
-    length="0.22"
-    mass="0.5"
-    material="Gazebo/Gold"
-    parent="base_link"
-    joint_origin_xyz="-0.0375 -0.1 0.185"
-  />
-  <xacro:standoff name="standoff4"
-    radius="0.01"
-    length="0.22"
-    mass="0.5"
-    material="Gazebo/Gold"
-    parent="base_link"
-    joint_origin_xyz="0.0375 -0.1 0.185"
-  />
-<!-- wheels -->
-  <xacro:wheel name="left_wheel"
-    radius="0.0352"
-    length="0.0206"
-    mass="0.5"
-    material="Gazebo/Green"
-    parent="base_link"
-    joint_origin_xyz="0 0.09 -0.05"
-  />
-  <xacro:wheel name="right_wheel"
-    radius="0.0352"
-    length="0.0206"
-    mass="0.5"
-    material="Gazebo/Green"
-    parent="base_link"
-    joint_origin_xyz="0 -0.09 -0.05"
-  />
-<!-- casters -->
-<!-- front caster -->
-  <link name="front_yaw_link">
-      <visual>
-        <origin rpy="0 1.5707 1.5707" xyz="0 0 0"/>
-        <geometry>
-          <cylinder length="0.01" radius="0.011"/>
-        </geometry>
-      </visual>
-      <collision>
-        <origin rpy="0 1.5707 1.5707" xyz="0 0 0"/>
-        <geometry>
-          <cylinder length="0.01" radius="0.01"/>
-        </geometry>
-      </collision>
-      <inertial>
-          <origin rpy="0 1.5707 1.5707" xyz="0 0 0"/>
-          <mass value="0.001"/>
-          <inertia ixx="5.145833333333334e-09" ixy="0" ixz="0" iyy="5.145833333333334e-09" iyz="0" izz="1.0125000000000003e-08"/>
-      </inertial>
-  </link>
-  <joint name="front_yaw_joint" type="continuous">
-    <origin rpy="0 0 0" xyz="0.15 0 -0.0753" />
-    <parent link="base_link" />
-    <child link="front_yaw_link" />
-    <axis xyz="0 0 1" />
-    <limit effort="1000.0" velocity="100.0" />
-    <dynamics damping="0.0" friction="0.1"/>
-  </joint>
-  <gazebo reference="front_yaw_link">
-    <kp>1000000000000000000000000000.0</kp>
-    <kd>1000000000000000000000000000.0</kd>
-    <mu1>0.5</mu1>
-    <mu2>0.5</mu2>
-  </gazebo>
-  <link name="front_roll_link">
-    <visual>
-      <origin rpy="0 1.5707 1.5707" xyz="0 0 0"/>
-      <geometry>
-        <cylinder length="0.01" radius="0.011"/>
-      </geometry>
-    </visual>
-    <collision>
-      <origin rpy="0 1.5707 1.5707" xyz="0 0 0"/>
-      <geometry>
-        <cylinder length="0.01" radius="0.011"/>
-      </geometry>
-    </collision>
-    <inertial>
-      <origin rpy="0 1.5707 1.5707" xyz="0 0 0"/>
-      <mass value="0.001"/>
-      <inertia ixx="5.145833333333334e-09" ixy="0" ixz="0" iyy="5.145833333333334e-09" iyz="0" izz="1.0125000000000003e-08"/>
-    </inertial>
-  </link>
-  <gazebo reference="front_roll_link">
-    <kp>1000000000000000000000000000.0</kp>
-    <kd>1000000000000000000000000000.0</kd>
-    <mu1>0.5</mu1>
-    <mu2>0.5</mu2>
-  </gazebo>
-  <joint name="front_roll_joint" type="continuous">
-    <origin rpy="0 0 0" xyz="0 0 0" />
-    <parent link="front_yaw_link" />
-    <child link="front_roll_link" />
-    <axis xyz="1 0 0" />
-    <limit effort="1000.0" velocity="100.0" />
-    <dynamics damping="0.0" friction="0.1"/>
-  </joint>
-  <link name="front_pitch_link">
-    <visual>
-      <origin rpy="0 1.5707 1.5707" xyz="0 0 0"/>
-      <geometry>
-        <sphere radius="0.010"/>
-      </geometry>
-    </visual>
-    <collision>
-      <origin rpy="0 1.5707 1.5707" xyz="0 0 0"/>
-      <geometry>
-        <sphere radius="0.010"/>
-      </geometry>
-    </collision>
-    <inertial>
-      <origin rpy="0 1.5707 1.5707" xyz="0 0 0"/>
-      <mass value="0.001"/>
-      <inertia ixx="4e-08" ixy="0" ixz="0" iyy="4e-08" iyz="0" izz="4e-08"/>
-    </inertial>
-  </link>
-  <gazebo reference="front_pitch_link">
-    <kp>1000000000000000000000000000.0</kp>
-    <kd>1000000000000000000000000000.0</kd>
-    <mu1>0.5</mu1>
-    <mu2>0.5</mu2>
-    <material>Gazebo/Purple</material>
-  </gazebo>
-  <joint name="front_pitch_joint" type="continuous">
-    <origin rpy="0 0 0" xyz="0 0 0" />
-    <parent link="front_roll_link" />
-    <child link="front_pitch_link" />
-    <axis xyz="0 1 0" />
-    <limit effort="1000.0" velocity="100.0" />
-    <dynamics damping="0.0" friction="0.1"/>
-  </joint>
-<!-- back caster -->
-  <link name="back_yaw_link">
-      <visual>
-        <origin rpy="0 1.5707 1.5707" xyz="0 0 0"/>
-        <geometry>
-          <cylinder length="0.01" radius="0.011"/>
-        </geometry>
-      </visual>
-      <collision>
-        <origin rpy="0 1.5707 1.5707" xyz="0 0 0"/>
-        <geometry>
-          <cylinder length="0.01" radius="0.011"/>
-        </geometry>
-      </collision>
-      <inertial>
-          <origin rpy="0 1.5707 1.5707" xyz="0 0 0"/>
-          <mass value="0.001"/>
-          <inertia ixx="5.145833333333334e-09" ixy="0" ixz="0" iyy="5.145833333333334e-09" iyz="0" izz="1.0125000000000003e-08"/>
-      </inertial>
-  </link>
-  <joint name="back_yaw_joint" type="continuous">
-    <origin rpy="0 0 0" xyz="-0.15 0 -0.0753" />
-    <parent link="base_link" />
-    <child link="back_yaw_link" />
-    <axis xyz="0 0 1" />
-    <limit effort="1000.0" velocity="100.0" />
-    <dynamics damping="0.0" friction="0.1"/>
-  </joint>
-    <gazebo reference="back_yaw_link">
-      <kp>1000000000000000000000000000.0</kp>
-      <kd>1000000000000000000000000000.0</kd>
-      <mu1>0.5</mu1>
-      <mu2>0.5</mu2>
-    </gazebo>
-  <link name="back_roll_link">
-      <visual>
-        <origin rpy="0 1.5707 1.5707" xyz="0 0 0"/>
-        <geometry>
-          <cylinder length="0.01" radius="0.011"/>
-        </geometry>
-      </visual>
-      <collision>
-        <origin rpy="0 1.5707 1.5707" xyz="0 0 0"/>
-        <geometry>
-          <cylinder length="0.01" radius="0.011"/>
-        </geometry>
-      </collision>
-      <inertial>
-          <origin rpy="0 1.5707 1.5707" xyz="0 0 0"/>
-          <mass value="0.001"/>
-          <inertia ixx="5.145833333333334e-09" ixy="0" ixz="0" iyy="5.145833333333334e-09" iyz="0" izz="1.0125000000000003e-08"/>
-      </inertial>
-  </link>
-  <joint name="back_roll_joint" type="continuous">
-    <origin rpy="0 0 0" xyz="0 0 0" />
-    <parent link="back_yaw_link" />
-    <child link="back_roll_link" />
-    <axis xyz="1 0 0" />
-    <limit effort="1000.0" velocity="100.0" />
-    <dynamics damping="0.0" friction="0.1"/>
-  </joint>
-    <gazebo reference="back_roll_link">
-      <kp>1000000000000000000000000000.0</kp>
-      <kd>1000000000000000000000000000.0</kd>
-      <mu1>0.5</mu1>
-      <mu2>0.5</mu2>
-    </gazebo>
-  <link name="back_pitch_link">
-    <visual>
-      <origin rpy="0 1.5707 1.5707" xyz="0 0 0"/>
-      <geometry>
-        <sphere radius="0.010"/>
-      </geometry>
-    </visual>
-    <collision>
-      <origin rpy="0 1.5707 1.5707" xyz="0 0 0"/>
-      <geometry>
-        <sphere radius="0.010"/>
-      </geometry>
-    </collision>
-    <inertial>
-        <origin rpy="0 1.5707 1.5707" xyz="0 0 0"/>
-        <mass value="0.001"/>
-        <inertia ixx="4e-08" ixy="0" ixz="0" iyy="4e-08" iyz="0" izz="4e-08"/>
-    </inertial>
-  </link>
-  <gazebo reference="back_pitch_link">
-    <kp>1000000000000000000000000000.0</kp>
-    <kd>1000000000000000000000000000.0</kd>
-    <mu1>0.5</mu1>
-    <mu2>0.5</mu2>
-    <material>Gazebo/Purple</material>
-  </gazebo>
-  <joint name="back_pitch_joint" type="continuous">
-    <origin rpy="0 0 0" xyz="0 0 0" />
-    <parent link="back_roll_link" />
-    <child link="back_pitch_link" />
-    <axis xyz="0 1 0" />
-    <limit effort="1000.0" velocity="100.0" />
-    <dynamics damping="0.0" friction="0.1"/>
-  </joint>
-<!-- drink tray -->
-  <xacro:cup_holder_tray name="drink_tray"
-    radius="0.16"
-    length="0.09"
-    mass="0.5"
-    material="Gazebo/Red"
-    parent="standoff1"
-    joint_origin_xyz="-0.035 -0.1 0.15"
-  />
-<!-- laser scanner -->
-  <xacro:laser_scanner>
-    <xacro:arg name="include_laser" value="${include_laser}" default="" />
-  </xacro:laser_scanner>
-  <!-- PLUGINS -->
-  <!-- JOINT PUBLISHER -->
-  <gazebo>
-    <plugin name="barista_robot_joint_state" filename="libgazebo_ros_joint_state_publisher.so">
-      <ros>
-          <remapping>~/out:=joint_states</remapping>
-      </ros>
-      <update_rate>30</update_rate>
-      <joint_name>left_wheel_joint</joint_name>
-      <joint_name>right_wheel_joint</joint_name>
-      <joint_name>front_yaw_joint</joint_name>
-      <joint_name>back_yaw_joint</joint_name>
-      <joint_name>front_roll_joint</joint_name>
-      <joint_name>back_roll_joint</joint_name>
-      <joint_name>front_pitch_joint</joint_name>
-      <joint_name>back_pitch_joint</joint_name>
-    </plugin>
-  </gazebo>
-  <!-- Differential drive -->
-  <gazebo>
-    <plugin filename="libgazebo_ros_diff_drive.so" name="differential_drive_controller">
-      <!-- wheels -->
-      <left_joint>left_wheel_joint</left_joint>
-      <right_joint>right_wheel_joint</right_joint>
-      <!-- kinematics -->
-      <wheel_separation>0.1</wheel_separation>
-      <wheel_diameter>0.07</wheel_diameter>
-      <!-- limits -->
-      <max_wheel_torque>1.0</max_wheel_torque>
-      <max_wheel_acceleration>2.0</max_wheel_acceleration>
-      <!-- output -->
-      <publish_odom>true</publish_odom>
-      <publish_odom_tf>true</publish_odom_tf>
-      <odometry_frame>odom</odometry_frame>
-      <robot_base_frame>base_link</robot_base_frame>
-    </plugin>
-  </gazebo>
-  <!-- Position Config -->
-  <ros2_control name="GazeboSystem" type="system">
-    <hardware>
-      <plugin>gazebo_ros2_control/GazeboSystem</plugin>
-    </hardware>
-    <joint name="hokuyo_joint">
-      <command_interface name="position">
-        <param name="min">-0.05</param>
-        <param name="max">0.0</param>
-      </command_interface>
-      <state_interface name="position"/>
-      <state_interface name="velocity"/>
-      <state_interface name="effort"/>
-    </joint>
-  </ros2_control>
-  <gazebo>
-    <plugin filename="libgazebo_ros2_control.so" name="gazebo_ros2_control">
-      <parameters>$(find barista_robot_description)/config/controller_position_velocity.yaml</parameters>
-      <robot_param_node>/my_robot_state_publisher_node</robot_param_node>
-    </plugin>
-  </gazebo>
+<xacro:base-plate
+    name = "base"
+    parent = "odom"
+    joint_origin_xyz = "0 0 0.0445"
+/>
+<xacro:standoff
+    name ="standoff1"
+    radius = "0.0025"
+    length = "0.0393"
+    mass = "0.5"
+    parent = "base_link"
+    joint_origin_xyz = "-0.06277 0.042975 0.01975"
+/>
+<xacro:standoff
+    name ="standoff2"
+    radius = "0.0025"
+    length = "0.0393"
+    mass = "0.5"
+    parent = "base_link"
+    joint_origin_xyz = "0.06277 0.042975 0.01975"
+/>
+<xacro:standoff
+    name ="standoff3"
+    radius = "0.0025"
+    length = "0.0393"
+    mass = "0.5"
+    parent = "base_link"
+    joint_origin_xyz = "0.06277 -0.042975 0.01975"
+/>
+<xacro:standoff
+    name ="standoff4"
+    radius = "0.0025"
+    length = "0.0393"
+    mass = "0.5"
+    parent = "base_link"
+    joint_origin_xyz = "-0.06277 -0.042975 0.01975"
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