Commit message: feat: setting correct mass values and refactoring the launch file

File: xacro/base-plate.xacro (robot description, xacro)
@@ -14,5 +14,5 @@
         </collision>
         <inertial>
-          <mass value="0.5"/>
+          <mass value="0.035"/>
           <origin rpy="0 0 0" xyz="0 0 0"/>
           <inertia ixx="0.0008333333333333335" ixy="0" ixz="0" iyy="0.0008333333333333335" iyz="0" izz="0.0008333333333333335"/>

File: xacro/camera.xacro (robot description, xacro)
@@ -18,5 +18,5 @@
             </collision>
             <inertial>
-                <mass value="0.05"/>
+                <mass value="0.001"/>
                 <origin xyz="0 0 0" rpy="0 0 0"/>
                 <inertia ixx="0.00001" ixy="0.0" ixz="0.0" iyy="0.00001" iyz="0.0" izz="0.00001"/>
@@ -33,5 +33,5 @@
         <link name="${name}_camera_bottom_link">
             <inertial>
-                <mass value="0.1"/>
+                <mass value="0.003"/>
                 <inertia ixx="0.001" ixy="0.0" ixz="0.0" iyy="0.001" iyz="0.0" izz="0.001"/>
             </inertial>
@@ -57,5 +57,5 @@
         <link name="${name}_camera_top_link">
             <inertial>
-                <mass value="0.1"/>
+                <mass value="0.003"/>
                 <inertia ixx="0.001" ixy="0.0" ixz="0.0" iyy="0.001" iyz="0.0" izz="0.001"/>
             </inertial>

File: xacro/imu.xacro (robot description, xacro)
@@ -17,5 +17,5 @@
             </collision>
             <inertial>
-                <mass value="0.02"/>
+                <mass value="0.002"/>
                 <origin xyz="0 0 0" rpy="0 0 0"/>
                 <inertia ixx="0.00001" ixy="0.0" ixz="0.0" iyy="0.00001" iyz="0.0" izz="0.00001"/>

File: xacro/my-jetbot.xacro (robot description, xacro)
@@ -5,5 +5,5 @@
     <xacro:include filename="$(find jetbot_sim)/xacro/base-plate.xacro"/>
     <xacro:include filename="$(find jetbot_sim)/xacro/ydlidar.xacro"/>
-    <xacro:include filename="$(find jetbot_sim)/xacro/camera.xacro"/>
+    <xacro:include filename="$(find jetb3ot_sim)/xacro/camera.xacro"/>
     <xacro:include filename="$(find jetbot_sim)/xacro/imu.xacro"/>
     <xacro:include filename="$(find jetbot_sim)/xacro/reflectance-sensor.xacro"/>
@@ -20,5 +20,5 @@
         radius = "0.0025"
         length = "0.0393"
-        mass = "0.5"
+        mass = "0.008"
         parent = "base_link"
         joint_origin_xyz = "-0.06277 0.042975 0.01975"
@@ -28,5 +28,5 @@
         radius = "0.0025"
         length = "0.0393"
-        mass = "0.5"
+        mass = "0.008"
         parent = "base_link"
         joint_origin_xyz = "0.06277 0.042975 0.01975"
@@ -36,5 +36,5 @@
         radius = "0.0025"
         length = "0.0393"
-        mass = "0.5"
+        mass = "0.008"
         parent = "base_link"
         joint_origin_xyz = "0.06277 -0.042975 0.01975"
@@ -44,5 +44,5 @@
         radius = "0.0025"
         length = "0.0393"
-        mass = "0.5"
+        mass = "0.008"
         parent = "base_link"
         joint_origin_xyz = "-0.06277 -0.042975 0.01975"
@@ -58,5 +58,5 @@
         radius = "0.0025"
         length = "0.081"
-        mass = "0.5"
+        mass = "0.016"
         parent = "level2_link"
         joint_origin_xyz = "-0.06277 0.042975 0.01975"
@@ -66,5 +66,5 @@
         radius = "0.0025"
         length = "0.081"
-        mass = "0.5"
+        mass = "0.016"
         parent = "level2_link"
         joint_origin_xyz = "0.06277 0.042975 0.01975"
@@ -74,5 +74,5 @@
         radius = "0.0025"
         length = "0.081"
-        mass = "0.5"
+        mass = "0.016"
         parent = "level2_link"
         joint_origin_xyz = "0.06277 -0.042975 0.01975"
@@ -82,5 +82,5 @@
         radius = "0.0025"
         length = "0.081"
-        mass = "0.5"
+        mass = "0.016"
         parent = "level2_link"
         joint_origin_xyz = "-0.06277 -0.042975 0.01975"
@@ -106,5 +106,5 @@
         radius = "0.0025"
         length = "0.023"
-        mass = "0.1"
+        mass = "0.004"
         parent = "base_link"
         joint_origin_xyz = "-0.05477 0.02 -0.01375"
@@ -114,5 +114,5 @@
         radius = "0.0025"
         length = "0.023"
-        mass = "0.1"
+        mass = "0.004"
         parent = "base_link"
         joint_origin_xyz = "-0.05477 -0.02 -0.01375"
@@ -130,5 +130,5 @@
         </collision>
         <inertial>
-          <mass value="0.5"/>
+          <mass value="0.003"/>
           <origin rpy="0 0 0" xyz="0 0 0"/>
           <inertia ixx="0.0008333333333333335" ixy="0" ixz="0" iyy="0.0008333333333333335" iyz="0" izz="0.0008333333333333335"/>
@@ -157,5 +157,5 @@
         </collision>
         <inertial>
-          <mass value="0.01"/>
+          <mass value="0.015"/>
           <origin xyz="0 0 0" rpy="0 0 0"/>
           <inertia ixx="0.00001" ixy="0.0" ixz="0.0" iyy="0.00001" iyz="0.0" izz="0.00001"/>
@@ -187,5 +187,5 @@
         radius = "0.0025"
         length = "0.033"
-        mass = "0.1"
+        mass = "0.006"
         parent = "level3_link"
         joint_origin_xyz = "-0.025 -0.0315 0.018"
@@ -195,5 +195,5 @@
         radius = "0.0025"
         length = "0.033"
-        mass = "0.1"
+        mass = "0.006"
         parent = "level3_link"
         joint_origin_xyz = "-0.025 0.0315 0.018"
@@ -203,5 +203,5 @@
         radius = "0.0025"
         length = "0.033"
-        mass = "0.1"
+        mass = "0.006"
         parent = "level3_link"
         joint_origin_xyz = "0.035 -0.0315 0.018"
@@ -211,5 +211,5 @@
         radius = "0.0025"
         length = "0.033"
-        mass = "0.1"
+        mass = "0.006"
         parent = "level3_link"
         joint_origin_xyz = "0.035 0.0315 0.018"
@@ -232,5 +232,5 @@
         </collision>
         <inertial>
-          <mass value="0.5"/>
+          <mass value="0.008"/>
           <origin rpy="0 0 0" xyz="0 0 0"/>
           <inertia ixx="0.0008333333333333335" ixy="0" ixz="0" iyy="0.0008333333333333335" iyz="0" izz="0.0008333333333333335"/>
@@ -255,5 +255,5 @@
             radius = "0.0025"
             length = "0.01"
-            mass = "0.5"
+            mass = "0.002"
             parent = "level3_link"
             joint_origin_xyz = "0.0275 -0.04 0.0065"
@@ -262,5 +262,5 @@
             name ="standoff16"
             radius = "0.0025"
-            length = "0.01"
+            length = "0.002"
             mass = "0.5"
             parent = "level3_link"
@@ -278,55 +278,57 @@
         joint_origin_xyz = "-0.01 0.014 -0.002"
     />
-    <!-- PLUGINS -->
-  <!-- JOINT PUBLISHER -->
-  <gazebo>
-    <plugin name="jetbot_joint_state" filename="libgazebo_ros_joint_state_publisher.so">
-      <update_rate>30</update_rate>
-      <joint_name>left_wheel_joint</joint_name>
-      <joint_name>right_wheel_joint</joint_name>
-      <joint_name>caster_ball_yaw_joint</joint_name>
-      <joint_name>caster_ball_roll_joint</joint_name>
-      <joint_name>caster_ball_pitch_joint</joint_name>
-    </plugin>
-  </gazebo>
-  <!-- Differential drive -->
-  <gazebo>
-    <plugin filename="libgazebo_ros_diff_drive.so" name="differential_drive_controller">
-      <!-- wheels -->
-      <left_joint>left_wheel_joint</left_joint>
-      <right_joint>right_wheel_joint</right_joint>
-      <!-- kinematics -->
-      <wheel_separation>0.13</wheel_separation>
-      <wheel_diameter>0.065</wheel_diameter>
-      <!-- limits -->
-      <max_wheel_torque>1.0</max_wheel_torque>
-      <max_wheel_acceleration>2.0</max_wheel_acceleration>
-      <!-- output -->
-      <publish_odom>true</publish_odom>
-      <publish_odom_tf>true</publish_odom_tf>
-      <odometry_frame>odom</odometry_frame>
-      <robot_base_frame>base_link</robot_base_frame>
-    </plugin>
-  </gazebo>
-  <!-- Position Config -->
-  <ros2_control name="GazeboSystem" type="system">
-    <hardware>
-      <plugin>gazebo_ros2_control/GazeboSystem</plugin>
-    </hardware>
-    <joint name="default_ydlidar_top_joint">
-      <command_interface name="position">
-        <param name="min">-0.05</param>
-        <param name="max">0.0</param>
-      </command_interface>
-      <state_interface name="position"/>
-      <state_interface name="velocity"/>
-      <state_interface name="effort"/>
-    </joint>
-  </ros2_control>
-  <gazebo>
-    <plugin filename="libgazebo_ros2_control.so" name="gazebo_ros2_control">
-      <parameters>$(find jetbot_sim)/config/controller_position_velocity.yaml</parameters>
-      <robot_param_node>robot_state_publisher</robot_param_node>
-    </plugin>
-  </gazebo>
+<!-- PLUGINS -->
+<!-- JOINT PUBLISHER -->
+<gazebo>
+  <plugin name="jetbot_joint_state" filename="libgazebo_ros_joint_state_publisher.so">
+    <update_rate>30</update_rate>
+    <joint_name>left_wheel_joint</joint_name>
+    <joint_name>right_wheel_joint</joint_name>
+    <joint_name>caster_ball_yaw_joint</joint_name>
+    <joint_name>caster_ball_roll_joint</joint_name>
+    <joint_name>caster_ball_pitch_joint</joint_name>
+  </plugin>
+</gazebo>
+<!-- Differential drive -->
+<gazebo>
+  <plugin filename="libgazebo_ros_diff_drive.so" name="differential_drive_controller">
+    <!-- wheels -->
+    <left_joint>left_wheel_joint</left_joint>
+    <right_joint>right_wheel_joint</right_joint>
+    <!-- kinematics -->
+    <wheel_separation>0.13</wheel_separation>
+    <wheel_diameter>0.065</wheel_diameter>
+    <!-- limits -->
+    <max_wheel_torque>1.0</max_wheel_torque>
+    <max_wheel_acceleration>2.0</max_wheel_acceleration>
+    <!-- output -->
+    <publish_odom>true</publish_odom>
+    <publish_odom_tf>true</publish_odom_tf>
+    <odometry_frame>odom</odometry_frame>
+    <robot_base_frame>base_link</robot_base_frame>
+    <!-- cmd_vel topic -->
+    <command_topic>/cmd_vel</command_topic>
+  </plugin>
+</gazebo>
+<!-- Position Config -->
+<ros2_control name="GazeboSystem" type="system">
+  <hardware>
+    <plugin>gazebo_ros2_control/GazeboSystem</plugin>
+  </hardware>
+  <joint name="default_ydlidar_top_joint">
+    <command_interface name="position">
+      <param name="min">-0.05</param>
+      <param name="max">0.0</param>
+    </command_interface>
+    <state_interface name="position"/>
+    <state_interface name="velocity"/>
+    <state_interface name="effort"/>
+  </joint>
+</ros2_control>
+<gazebo>
+  <plugin filename="libgazebo_ros2_control.so" name="gazebo_ros2_control">
+    <parameters>$(find jetbot_sim)/config/controller_position_velocity.yaml</parameters>
+    <robot_param_node>robot_state_publisher</robot_param_node>
+  </plugin>
+</gazebo>
 </robot>

File: xacro/reflectance-sensor.xacro (robot description, xacro)
@@ -16,5 +16,5 @@
             </collision>
             <inertial>
-                <mass value="0.05"/>
+                <mass value="0.002"/>
                 <origin xyz="0 0 0" rpy="0 0 0"/>
                 <inertia ixx="0.00001" ixy="0.0" ixz="0.0" iyy="0.00001" iyz="0.0" izz="0.00001"/>

File: xacro/wheel.xacro (robot description, xacro)
@@ -5,5 +5,5 @@
             <inertial>
                 <origin rpy="0 1.5707 1.5707" xyz="0 0 0"/>
-                <mass value="0.1"/>
+                <mass value="0.065"/>
                 <inertia ixx="0.001" ixy="0.0" ixz="0.0" iyy="0.001" iyz="0.0" izz="0.001"/>
             </inertial>

File: xacro/ydlidar.xacro (robot description, xacro)
@@ -14,5 +14,5 @@
         </collision>
         <inertial>
-          <mass value="0.5"/>
+          <mass value="0.023"/>
           <origin rpy="0 0 0" xyz="0 0 0"/>
           <inertia ixx="0.0008333333333333335" ixy="0" ixz="0" iyy="0.0008333333333333335" iyz="0" izz="0.0008333333333333335"/>
@@ -29,5 +29,5 @@
       <link name="${name}_ydlidar_top_link">
         <inertial>
-          <mass value="0.1"/>
+          <mass value="0.023"/>
           <inertia ixx="0.001" ixy="0.0" ixz="0.0" iyy="0.001" iyz="0.0" izz="0.001"/>
         </inertial>
@@ -53,5 +53,5 @@
       <link name="${name}_ydlidar_motor_link">
         <inertial>
-          <mass value="0.1"/>
+          <mass value="0.024"/>
           <inertia ixx="0.001" ixy="0.0" ixz="0.0" iyy="0.001" iyz="0.0" izz="0.001"/>
         </inertial>
